File: DroneSchematic.kicad_sch (KiCad schematic)
At the start: 0 parts

Commit message: july 28 make sure everything is up to date in the master
Parts:
- added A?: FrSky_X8R, symbol DroneSchematicLib:FrSky_X8R
- added A?: Wifi_module, symbol DroneSchematicLib:Wifi_module
- added BT?: Glacier_6s_3300mah, symbol DroneSchematicLib:Glacier_6s_3300mah
- added M? (x4): Tmotor_v2207, symbol DroneSchematicLib:Tmotor_v2207
- added U?: OpticalFlow, symbol DroneSchematicLib:OpticalFlow
- added U?: UBEC, symbol DroneSchematicLib:UBEC
- added U?: HolyBroTekkoEsc, symbol DroneSchematicLib:HolyBroTekkoEsc
- added U?: HolyBro_Kakute_H7_BT, symbol DroneSchematicLib:HolyBro_Kakute_H7_BT
- added U?: ToF_IR, symbol DroneSchematicLib:ToF_IR
- added U?: UP_board, symbol DroneSchematicLib:UP_board
Connections:
- new net: M?. (Phase_3), U?. (Vbat) (x12)
- new net: U?. (Vcc), U?. (Vdd) (x7)
- new net: BT?. (V_cell6), U?. (GND), U?. (Vbat), U?.7 (Vbat)
- new net: BT?. (V_cell6), U?. (GND), U?. (Vbat), U?.8 (GND)
- new net: U?. (GND), U?. (Vdd) (x2)
- new net: U?. (Vbat), U?.10 (M2)
- new net: U?. (Vbat), U?.11 (M3)
- new net: U?. (Vbat), U?.12 (M4)
- new net: U?. (Vbat), U?.13 (Vbat_monitor)
- new net: U?. (Vbat), U?.14 (TLM)
- new net: U?. (Vbat), U?.15 (GND)
- new net: U?. (Vbat), U?.16 (I_monitor)
- new net: U?. (Vbat), U?.9 (M1)
- new net: U?. (Vdd), U?.1 (T3)
- new net: U?. (Vdd), U?.2 (R3)
- new net: A?. (SBus_Vdd), U?.3 (T6)
- new net: A?. (SBus_Vdd), U?.4 (R4)
- new net: A?. (SBus_Vdd), U?.5 (Vdd)
- new net: A?. (SBus_Vdd), U?.6 (GND)
- new net: U?. (Vdd), U?. (Vdd) (x4)
- new net: A?. (BT/WIFI_y), U?. (Vdd)
